File: AT24-Timer-Polair/AT24-Timer.brd (EAGLE design)
At the start: 100 x 90.2 mm, 66 parts, among them Q1 SI2302, Q2 SI2302, Q3 SI2302, Q4 SI2302, Q5 SI2302, T1 BT136, U1 DS3231, U2 ATTINY24A-SU, U3 XL1530, U4 74HC595D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

Commit message: Добавлены ДХО работающие на ШИМ
Parts:
- added R29: S14K300, varistor:S14K300
- R10: value 1k -> 1k5
- R9: value 1.3k -> 1k
- moved R27 214.3 mm to (74.9, 42.4), flipped to the bottom, turned to 270 degrees
- moved R28 208.3 mm to (71.1, 30.0), flipped to the bottom, turned to 180 degrees
- moved R26 191.6 mm to (63.5, 30.3), flipped to the bottom, turned to 270 degrees
- moved R25 185.4 mm to (71.1, 25.4), flipped to the bottom, turned to 180 degrees
- moved R20 181.1 mm to (71.1, 27.6), flipped to the bottom, turned to 180 degrees
- moved R19 180.2 mm to (71.4, 33.8), flipped to the bottom, turned to 270 degrees
- moved S3 176.6 mm to (85.9, 44.5), turned to 90 degrees
- moved R18 171.9 mm to (61.0, 38.9), flipped to the bottom
- moved R17 162.0 mm to (65.7, 30.3), flipped to the bottom, turned to 270 degrees
- moved R4 136.7 mm to (19.7, 41.8), flipped to the bottom, turned to 270 degrees
- moved X5 132.8 mm to (80.2, 6.83)
- moved JP1 124.2 mm to (13.3, 38.3)
- moved U1 102.1 mm to (37.1, 17.9), flipped to the bottom, turned to 180 degrees
- moved C11 90.6 mm to (9.21, 25.6), turned to 270 degrees
- moved L1 86.5 mm to (23.2, 31.6), flipped to the bottom, turned to 270 degrees
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Connections:
- removed net N$26: R10.2, R9.2, S1.3, S1.4
- new net N$160: R10.2, R9.2, S2.3, S2.4
- net N$1: now also R29.1
- net N$14: now also R29.2
- net N$6: now also S1.3, S1.4; no longer S2.3, S2.4
Routing:
- net GND: track 66.7 -> 294.1 mm, vias 4 -> 0
- net GND1: track 2.00 -> 136.6 mm, vias 0 -> 2
- net VCC: track 30.2 -> 140.9 mm, vias 0 -> 2
- net VCC/2: track 6.02 -> 99.8 mm, vias 0 -> 2
- net N$11: track 0.00 -> 70.8 mm, vias 0 -> 2
- net N$21: track 0.00 -> 30.5 mm
- net N$10: track 47.9 -> 17.5 mm
- net N$4: track 66.5 -> 37.0 mm, vias 2 -> 0
- net N$5: track 61.7 -> 33.7 mm
- net N$40: track 4.84 -> 29.1 mm
- net N$30: track 50.9 -> 71.7 mm, vias 2 -> 0
- net N$23: track 0.00 -> 20.2 mm, vias 0 -> 2
- net N$65: track 25.3 -> 5.29 mm
- net N$53: track 0.00 -> 17.8 mm
- net N$42: track 3.67 -> 19.1 mm
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Other:
- board size 100 x 90.2 mm -> 100.3 x 79.7 mm
- board text added: "2016"
- board text added: "zzzMariKzzz"
- board text added: "zzzMariKzzz 2016"
- board text removed: "Menu"
- board text removed: "OK"
- board text removed: "Simple Timer"
- board text removed: "zzzMariKzzz 2015"
