File: AT24-Timer-Polair/AT24-Timer.sch (EAGLE design)
At the start: 66 parts, among them Q1 SI2302, Q2 SI2302, Q3 SI2302, Q4 SI2302, Q5 SI2302, T1 BT136, U1 DS3231, U2 ATTINY24A-SU, U3 XL1530, U4 74HC595D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

Commit message: Добавлены ДХО работающие на ШИМ
Parts:
- added R29: S14K300, varistor:S14K300
- R10: value 1k -> 1k5
- R9: value 1.3k -> 1k
Connections:
- removed net N$26: R10.2, R9.2, S1.3, S1.4
- removed net N$50: R9.1, S3.3, S3.4
- new net N$16: R9.1, S3.2
- new net N$160: R10.2, R9.2, S2.2
- net GND1: no longer S1.2, S2.2, S3.2
- net N$1: now also R29.1
- net N$14: now also R29.2
- net N$6: now also S1.2; no longer S2.3, S2.4
Other:
- note added: ""62""
- note added: ""86""
- note removed: ""45""
- note removed: ""84""
- moved on the sheet: R9
