File: Fog_DRL_Cam/Fog_DRL_Cam.sch (EAGLE design)
At the start: 51 parts, among them IC1 78L05Z, IC2 TINY13-20SSU, IC3 TINY13-20SSU, K1 CQ1-12V, K2 CQ1-12V, Q1 SI2302, X1 RCAX2, X10 PROG-ISP6POGOPIN, X11 PROG-ISP6POGOPIN, X2 PS/2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

Commit message: Добавлены ДХО работающие на ШИМ
Parts:
- removed C3: (no value), rcl:C-EUC0603
- removed H1: Reverse, holes:MOUNT-HOLE2.8
- removed H6: Bliz, holes:MOUNT-HOLE2.8
- removed H7: +12V, holes:MOUNT-HOLE3.0
- removed H8: GND, holes:MOUNT-HOLE3.0
- removed H9: Mar, holes:MOUNT-HOLE2.8
- removed IC2, IC3: TINY13-20SSU, atmel:TINY13-20SSU
- removed X10, X11: PROG-ISP6POGOPIN, usb:PROG-ISP6POGOPIN
- removed X4, X7, X8, X9: JST2, usb:JST2
- removed X5, X6: USB-FEMALE, usb:USB-FEMALE
- added C6, C7: 22pF, rcl:C-EUC0603
- added D5: (no value), diode:ZENER-DIODESOD80C
- added Q2: 16MHz, crystal:CRYSTALHC49S
- added R13: 10k, rcl:R-EU_R0603
- added U1: ATTINY24A-SU, usb:ATTINY24A-SU
- C4: value (none) -> 100n
- IC1: value 78L05Z -> 78L05F; device linear:78L05Z -> linear:78L05F
- Q1: value SI2302 -> IRLML2502
- R6: value 10k -> 2k2
- X1: value RCAX2 -> PROG-ISP6POGOPIN; device usb:RCAX2 -> usb:PROG-ISP6POGOPIN
- X3: value JST2 -> MOLEX18; device usb:JST2 -> usb:MOLEX18
Connections:
- removed net N$10: X6.D+, X6.D-
- removed net N$23: IC2.PB5/PCINT5/!RESET!/ADC0/DW, R6.1, X11.RST
- removed net N$24: IC2.PB0/PCINT0/AIN0/OC0A/MOSI, R8.1, X11.MOSI
- removed net N$29: IC3.PB0/PCINT0/AIN0/OC0A/MOSI, R10.1, X10.MOSI
- removed net N$30: IC3.PB1/PCINT1/AIN1/OC0B/INT0/MISO, R11.2, X10.MISO, X2.1
- removed net N$9: X5.D+, X5.D-
- new net CAM_RELAY: R10.1, U1.(ADC5/DO/MISO/OC1B/PCINT5)PA5, X1.MISO
- new net MAR: D5.C, R13.1, R6.1, U1.(ADC3/T0/PCINT3)PA3
- new net N$38: R9.2, U1.PB3(RESET/DW), X1.RST
- new net N$39: C7.1, Q2.2, U1.PB1(XTAL2)
- new net REVERS_KEY: R11.2, U1.(ADC6/DI/MOSI/SDA/OC1A/PCINT6)PA6, X1.MOSI, X2.1
- net +12V: now also X3.P$17; no longer X3.+, X4.+
- net +5V: now also U1.VCC, X1.VCC; no longer C3.1, IC2.VCC, IC3.VCC, R6.2, X10.VCC, X11.VCC
- net BLIZHNIY: now also U1.(ADC4/USCK/SCL/T1/PCINT4)PA4, X1.SCK; no longer IC2.PB3/PCINT3/CLKI/ADC3
- net GND: now also C6.2, C7.2, D5.A, IC1.GND@1, R13.2, U1.GND, VT1.E, X1.GND, X2.GND2, X3.P$15, X3.P$5; no longer C3.2, H8.P$1, IC2.GND, IC3.GND, VT1.C, X10.GND, X11.GND, X3.-, X4.-
- net N$1: now also X3.P$16; no longer X1.AV1
- net N$11: now also X3.P$4; no longer X7.+
- net N$12: now also X3.P$3; no longer X7.-
- net N$13: now also R6.2, X3.P$2; no longer H9.P$1
- net N$14: now also U1.(ADC7/ICP/OC0B/PCINT7)PA7; no longer IC2.PB4/PCINT4/ADC2
- net N$15: now also X3.P$13; no longer X8.-
- net N$16: now also X3.P$12; no longer X8.+
- net N$17: now also R8.1, U1.(ADC1/AIN0/PCINT1)PA1; no longer IC2.PB1/PCINT1/AIN1/OC0B/INT0/MISO, R7.1, X11.MISO
- net N$18: now also R7.1, U1.(ADC0/AREF/PCINT0)PA0; no longer IC3.PB2/PCINT2/SCK/ADC1/T0, X10.SCK
- net N$19: now also U1.(ADC2/AIN1/PCINT2)PA2, X3.P$10; no longer IC2.PB2/PCINT2/SCK/ADC1/T0, X11.SCK, X9.+
- net N$2: now also X3.P$11; no longer X9.-
- net N$21: now also X3.P$9; no longer H1.P$1
- net N$22: now also X3.P$6; no longer H6.P$1
- net N$27: now also C6.1, Q2.1, U1.PB0(XTAL1/CLKI); no longer IC3.PB5/PCINT5/!RESET!/ADC0/DW, R9.2, X10.RST
- net N$3: now also X3.P$14; no longer X1.GND1, X1.GND2
- net N$31: now also X3.P$18; no longer X1.AV2
- net N$5: now also VT1.C; no longer VT1.E
- net N$6: now also X3.P$1; no longer H7.P$1
- net N$7: now also X3.P$8; no longer X5.VCC, X6.VCC
- net N$8: now also X3.P$7; no longer X5.GND, X5.GND@1, X5.GND@2, X6.GND, X6.GND@1, X6.GND@2
- net REVERSE: now also U1.(CKOUT/OC0A/INT0)PB2; no longer IC3.PB3/PCINT3/CLKI/ADC3
Other:
- note added: "+12"
- note added: "Back Cam"
- note added: "Cam GND"
- note added: "Cam PW"
- note added: "GND"
- note added: "Key"
- note added: "MAR"
- note added: "Side Cam"
- note added: "USB PW"
- note removed: "Pri aktivacii +"
- note removed: "Pri aktivacii -"
- moved on the sheet: C4, D3, D4, R4, R5, R6, R8, R9, VT1
