File: AT24-Timer/AT24-Timer.brd (EAGLE design)
At the start: 100 x 49.7 mm, 51 parts, among them Q1 SI2302, Q2 SI2302, Q3 SI2302, Q4 SI2302, Q5 SI2302, T1 BT136, U1 DS1307, U2 ATTINY24A-SU, U4 74HC595D, U5 74HC595D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

Commit message: add
Parts:
- R12: value 470 -> 4k7
- R13: value 360 -> 3k
